File: gate-pcb/gate-pcb.kicad_pcb (KiCad board)
At the start: 2 copper layers, 21 x 25.5 mm, 6 parts, among them J1 EXT_IN, J2 EXT_OUT, J3 LED_START, J4 LED_END

Commit message: v1
Parts:
- moved REF** 18.0 mm to (124.8, 53.2)
- moved J2 2.06 mm to (107.5, 51.5)
- moved J4 2.06 mm to (123.0, 36.0)
- moved J1 0.71 mm to (107.5, 42.5)
- moved J3 0.71 mm to (114.0, 36.0)
- moved REF** 0.35 mm to (107.2, 35.8)
Routing:
- net Net-(J2-DATA_OUT): track 21.3 -> 25.4 mm
- net Net-(J1-DATA_IN): track 10.1 -> 11.5 mm
- net Net-(J1-GND): vias 16 -> 37
Other:
- board size 21 x 25.5 mm -> 23 x 23 mm

Commit message: fix backside 5v fill to connect with pads
Other:
- board text added: "Gate v2"
- board text removed: "Gate v1"
Changed lines of the file:
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@@
 		)
 	)
-	(gr_text "Gate v1"
+	(gr_text "Gate v2"
 		(at 116 55.5 0)
 		(layer "F.SilkS")
@@
 			(font
 				(size 1 1)
-				(thickness 0.15)
+				(thickness 0.2)
+				(bold yes)
 			)
 			(justify bottom)
@@
 		(net 3)
 		(net_name "Net-(J1-+5V)")
-		(layer "F.Cu")
+		(layers "F.Cu" "B.Cu")
 		(hatch edge 0.5)
 		(priority 1)
@@
 		(polygon
 			(pts
-				(xy 112 47.5) (xy 106.5 47.5) (xy 106.5 49.5) (xy 112 49.5)
+				(xy 112 47.5) (xy 106 47.5) (xy 106 49.5) (xy 112 49.5)
 			)
 		)
@@
 		(net 3)
 		(net_name "Net-(J1-+5V)")
-		(layer "F.Cu")
+		(layers "F.Cu" "B.Cu")
 		(hatch edge 0.5)
 		(priority 1)
@@
 		(polygon
 			(pts
-				(xy 112 35) (xy 110 35) (xy 110 40.5) (xy 112 40.5)
+				(xy 112 34.5) (xy 110 34.5) (xy 110 40.5) (xy 112 40.5)
 			)
 		)
 	)
 	(zone
-		(net 3)
-		(net_name "Net-(J1-+5V)")
-		(layer "F.Cu")
+		(net 2)
+		(net_name "Net-(J1-GND)")
+		(layers "F.Cu" "B.Cu")
 		(hatch edge 0.5)
 		(connect_pads yes
@@
 		(polygon
 			(pts
-				(xy 112 38.5) (xy 106.5 38.5) (xy 106.5 40.5) (xy 112 40.5)
+				(xy 127.5 33) (xy 104.5 33) (xy 104.5 56) (xy 127.5 56)
 			)
 		)
@@
 		(net 3)
 		(net_name "Net-(J1-+5V)")
-		(layer "F.Cu")
+		(layers "F.Cu" "B.Cu")
 		(hatch edge 0.5)
 		(connect_pads yes
@@
 		(polygon
 			(pts
-				(xy 121 35) (xy 119 35) (xy 119 40.5) (xy 121 40.5)
+				(xy 112 38.5) (xy 106 38.5) (xy 106 40.5) (xy 112 40.5)
 			)
 		)
 	)
 	(zone
-		(net 2)
-		(net_name "Net-(J1-GND)")
+		(net 3)
+		(net_name "Net-(J1-+5V)")
 		(layers "F.Cu" "B.Cu")
 		(hatch edge 0.5)
@@
 		(polygon
 			(pts
-				(xy 127.5 33) (xy 104.5 33) (xy 104.5 56) (xy 127.5 56)
+				(xy 121 34.5) (xy 119 34.5) (xy 119 40.5) (xy 121 40.5)
 			)
 		)
